File: TP_IVAN_LEON/Alimentacioon.sch (KiCad schematic (older format))
At the start: 5 parts, among them P1 POWER IN, U1 LM7805

Commit message: Acabado el pcb, aun no se agrega titulos a los sheets y falta completar cmapos de componenetes
Parts:
- removed U1: LM7805, symbol LM7805
- added U1: LM117H, TP:SOT-223, symbol LM117H
- added U5: LD1117S12TR, TP:SOT-223, symbol LD1117S12TR
- P1: footprint (none) -> TP:Connector_Molex_PicoBlade_53047-0210
Connections:
- net 3.3V: now also U5.2 (VO)
- net 5V: now also U1.3 (OUT), U5.3 (VI)
- net GND: now also U1.2 (ADJ), U5.1 (GND)
- net at C6.1, P1.2 (P2): now also U1.1 (IN)
Other:
- moved on the sheet: C6, P1
Changed lines of the file:
@@
 LIBS:MIproy1-cache
 LIBS:nxp_armmcu
+LIBS:DCV1_0-cach
 LIBS:DCV1_0-cache
 EELAYER 25 0
@@
 $EndDescr
 $Comp
-L LM7805 U1
-U 1 1 5782E47A
-P 4450 2750
-F 0 "U1" H 4600 2554 50  0000 C CNN
-F 1 "LM7805" H 4450 2950 50  0000 C CNN
-F 2 "" H 4450 2750 50  0001 C CNN
-F 3 "" H 4450 2750 50  0000 C CNN
-	1    4450 2750
-	1    0    0    -1
-$EndComp
-$Comp
-L AIC1117-33CY #U06
-U 1 1 5782E8B8
-P 5750 2700
-F 0 "#U06" H 5850 2400 60  0001 C CNN
-F 1 "AIC1117-33CY" H 5800 2850 60  0000 C CNN
-F 2 "" H 5750 2900 60  0000 C CNN
-F 3 "" H 5750 2900 60  0000 C CNN
-	1    5750 2700
-	1    0    0    -1
-$EndComp
-Wire Wire Line
-	4850 2700 5300 2700
-Wire Wire Line
-	4450 3000 4450 3250
-Wire Wire Line
-	5750 3100 5750 3250
-$Comp
-L GND #PWR07
+L GND #PWR06
 U 1 1 5784395E
 P 5100 3250
-F 0 "#PWR07" H 5100 3000 50  0001 C CNN
+F 0 "#PWR06" H 5100 3000 50  0001 C CNN
 F 1 "GND" H 5100 3100 50  0000 C CNN
 F 2 "" H 5100 3250 50  0000 C CNN
@@
 	1    0    0    -1
 $EndComp
-Wire Wire Line
-	3400 2700 4050 2700
-Wire Wire Line
-	6200 2700 6725 2700
 $Comp
 L Cap_1206 C7
@@
 L Cap_1206 C6
 U 1 1 5784480A
-P 3850 3000
-F 0 "C6" H 3850 2900 30  0000 C CNN
-F 1 "Cap_1206" H 3850 3075 30  0000 C CNN
-F 2 "TP:c_1206" H 3875 3000 60  0001 C CNN
-F 3 "" H 3875 3000 60  0000 C CNN
-	1    3850 3000
+P 3325 3000
+F 0 "C6" H 3325 2900 30  0000 C CNN
+F 1 "Cap_1206" H 3325 3075 30  0000 C CNN
+F 2 "TP:c_1206" H 3350 3000 60  0001 C CNN
+F 3 "" H 3350 3000 60  0000 C CNN
+	1    3325 3000
 	0    1    1    0
 $EndComp
-Connection ~ 3850 2700
+Connection ~ 3325 2700
 Wire Wire Line
-	3850 3125 3850 3250
-Connection ~ 4450 3250
+	3325 3125 3325 3250
 Wire Wire Line
 	4950 2825 4950 2700
@@
 	6350 3250 6350 3150
 Wire Wire Line
-	3400 3250 6350 3250
-Connection ~ 5750 3250
+	2875 3250 6350 3250
 Connection ~ 5100 3250
 $Comp
-L PWR_FLAG #FLG08
+L PWR_FLAG #FLG07
 U 1 1 5785C6B9
-P 3675 2625
-F 0 "#FLG08" H 3675 2720 50  0001 C CNN
-F 1 "PWR_FLAG" H 3675 2805 50  0000 C CNN
-F 2 "" H 3675 2625 50  0000 C CNN
-F 3 "" H 3675 2625 50  0000 C CNN
-	1    3675 2625
+P 3150 2625
+F 0 "#FLG07" H 3150 2720 50  0001 C CNN
+F 1 "PWR_FLAG" H 3150 2805 50  0000 C CNN
+F 2 "" H 3150 2625 50  0000 C CNN
+F 3 "" H 3150 2625 50  0000 C CNN
+	1    3150 2625
 	1    0    0    -1
 $EndComp
 Wire Wire Line
-	3675 2625 3675 2700
-Connection ~ 3675 2700
+	3150 2625 3150 2700
+Connection ~ 3150 2700
 Wire Wire Line
-	3850 2875 3850 2700
+	3325 2875 3325 2700
 $Comp
 L CONN_01X02 P1
 U 1 1 5798EC3A
-P 3200 2750
-F 0 "P1" H 3200 2900 50  0000 C CNN
-F 1 "POWER IN" V 3300 2750 50  0000 C CNN
-F 2 "" H 3200 2750 50  0001 C CNN
-F 3 "" H 3200 2750 50  0000 C CNN
-	1    3200 2750
+P 2675 2750
+F 0 "P1" H 2675 2900 50  0000 C CNN
+F 1 "POWER IN" V 2775 2750 50  0000 C CNN
+F 2 "TP:Connector_Molex_PicoBlade_53047-0210" H 2675 2750 50  0001 C CNN
+F 3 "" H 2675 2750 50  0000 C CNN
+	1    2675 2750
 	-1   0    0    1
 $EndComp
 Wire Wire Line
-	3400 2800 3400 3250
-Connection ~ 3850 3250
+	2875 2800 2875 3250
+Connection ~ 3325 3250
 Text GLabel 5100 2425 2    40   Output ~ 0
 5V
@@
 Wire Wire Line
 	6350 2700 6350 2900
+$Comp
+L LD1117S12TR U5
+U 1 1 57A6696E
+P 5775 2750
+F 0 "U5" H 5775 3000 50  0000 C CNN
+F 1 "LD1117S12TR" H 5775 2950 50  0000 C CNN
+F 2 "TP:SOT-223" H 5775 2850 50  0000 C CNN
+F 3 "" H 5775 2750 50  0000 C CNN
+	1    5775 2750
+	1    0    0    -1
+$EndComp
+Wire Wire Line
+	6175 2700 6725 2700
+Wire Wire Line
+	5775 3000 5775 3250
+Connection ~ 5775 3250
+Wire Wire Line
+	4625 2700 5375 2700
+Wire Wire Line
+	2875 2700 3825 2700
+Wire Wire Line
+	4225 3000 4225 3250
+Connection ~ 4225 3250
+$Comp
+L LM117H U1
+U 1 1 57A689CC
+P 4225 2750
+F 0 "U1" H 4025 2950 50  0000 C CNN
+F 1 "LM117H" H 4225 2950 50  0000 L CNN
+F 2 "TP:SOT-223" H 4225 2850 50  0000 C CIN
+F 3 "" H 4225 2750 50  0000 C CNN
+	1    4225 2750
+	1    0    0    -1
+$EndComp
 $EndSCHEMATC
