File: TP_IVAN_LEON/Alimentacioon.sch (KiCad schematic (older format))
At the start: 6 parts, among them P1 POWER IN, U1 LM117H, U5 LD1117S12TR

Commit message: Agregado codigo digey key en 80% de componentes
Parts:
- C6: value Cap_1206 -> 10uf; Digikey# (none) -> 490-6473-6-ND
- C7, C8: value Cap_1206 -> 1uf; Digikey# (none) -> 399-1254-2-ND
- P1: Digikey# (none) -> WM1731-ND
- U1: value LM117H -> 78L05; Digikey# (none) -> 497-1183-2-ND
- U5: Digikey# (none) -> 497-4240-2-ND
Changed lines of the file:
@@
 P 4950 2950
 F 0 "C7" H 4950 2850 30  0000 C CNN
-F 1 "Cap_1206" H 4950 3025 30  0000 C CNN
+F 1 "1uf" H 4950 3025 30  0000 C CNN
 F 2 "TP:c_1206" H 4975 2950 60  0001 C CNN
 F 3 "" H 4975 2950 60  0000 C CNN
+F 4 "399-1254-2-ND" H 4950 2950 60  0001 C CNN "Digikey#"
 	1    4950 2950
 	0    1    1    0
@@
 P 3325 3000
 F 0 "C6" H 3325 2900 30  0000 C CNN
-F 1 "Cap_1206" H 3325 3075 30  0000 C CNN
+F 1 "10uf" H 3325 3075 30  0000 C CNN
 F 2 "TP:c_1206" H 3350 3000 60  0001 C CNN
 F 3 "" H 3350 3000 60  0000 C CNN
+F 4 "490-6473-6-ND" H 3325 3000 60  0001 C CNN "Digikey#"
 	1    3325 3000
 	0    1    1    0
@@
 P 6350 3025
 F 0 "C8" H 6350 2925 30  0000 C CNN
-F 1 "Cap_1206" H 6350 3100 30  0000 C CNN
+F 1 "1uf" H 6350 3100 30  0000 C CNN
 F 2 "TP:c_1206" H 6375 3025 60  0001 C CNN
 F 3 "" H 6375 3025 60  0000 C CNN
+F 4 "399-1254-2-ND" H 6350 3025 60  0001 C CNN "Digikey#"
 	1    6350 3025
 	0    1    1    0
@@
 F 2 "TP:Connector_Molex_PicoBlade_53047-0210" H 2675 2750 50  0001 C CNN
 F 3 "" H 2675 2750 50  0000 C CNN
+F 4 "WM1731-ND" H 2675 2750 60  0001 C CNN "Digikey#"
 	1    2675 2750
 	-1   0    0    1
@@
 F 0 "U5" H 5775 3000 50  0000 C CNN
 F 1 "LD1117S12TR" H 5775 2950 50  0000 C CNN
-F 2 "TP:SOT-223" H 5775 2850 50  0000 C CNN
+F 2 "TP:SOT-223" H 5775 2850 50  0001 C CNN
 F 3 "" H 5775 2750 50  0000 C CNN
+F 4 "497-4240-2-ND" H 5775 2750 60  0001 C CNN "Digikey#"
 	1    5775 2750
 	1    0    0    -1
@@
 P 4225 2750
 F 0 "U1" H 4025 2950 50  0000 C CNN
-F 1 "LM117H" H 4225 2950 50  0000 L CNN
-F 2 "TP:SOT-223" H 4225 2850 50  0000 C CIN
+F 1 "78L05" H 4225 2950 50  0000 L CNN
+F 2 "TP:SOT-223" H 4225 2850 50  0001 C CIN
 F 3 "" H 4225 2750 50  0000 C CNN
+F 4 "497-1183-2-ND" H 4225 2750 60  0001 C CNN "Digikey#"
 	1    4225 2750
 	1    0    0    -1
