File: TP_IVAN_LEON/Entradas_Digitales.sch (KiCad schematic (older format))
At the start: 7 parts, among them J1 Teclado

Commit message: Acabado el pcb, aun no se agrega titulos a los sheets y falta completar cmapos de componenetes
Parts:
- J1: footprint (none) -> TP:Connector_Molex_PicoBlade_53047-0810
- R1: footprint (none) -> TP:Resistor_Array_SIP8
Changed lines of the file:
@@
 LIBS:MIproy1-cache
 LIBS:nxp_armmcu
+LIBS:DCV1_0-cach
 LIBS:DCV1_0-cache
 EELAYER 25 0
@@
 F 0 "J1" H 7800 3450 60  0000 C CNN
 F 1 "Teclado" H 7800 2700 60  0000 C CNN
-F 2 "" H 7750 3075 60  0001 C CNN
+F 2 "TP:Connector_Molex_PicoBlade_53047-0810" H 7750 3075 60  0001 C CNN
 F 3 "" H 7750 3075 60  0000 C CNN
 	1    7875 3075
@@
 F 0 "R1" H 4600 3200 60  0000 C CNN
 F 1 "Resistor_Array_10K" H 4550 2325 60  0000 C CNN
-F 2 "" H 4575 2875 60  0001 C CNN
+F 2 "TP:Resistor_Array_SIP8" H 4575 2875 60  0001 C CNN
 F 3 "" H 4575 2875 60  0000 C CNN
 	1    4650 2875
