File: TP_IVAN_LEON/LCD.sch (KiCad schematic (older format))
At the start: 4 parts, among them P2 CONN_02X08

Commit message: Acabado el pcb, aun no se agrega titulos a los sheets y falta completar cmapos de componenetes
Parts:
- P2: footprint (none) -> TP:Pin_Header_Straight_2x08
- R5: footprint TP:Resistor_SMD+THTuniversal_1206_RM10_HandSoldering_RevA_Date25Jun2010 -> TP:Resistor_SMD+THTuniversal_1206_RM10_HandSoldering
- RV1, RV2: footprint (none) -> TP:Connector_Molex_PicoBlade_53047-0310
Changed lines of the file:
@@
 LIBS:MIproy1-cache
 LIBS:nxp_armmcu
+LIBS:DCV1_0-cach
 LIBS:DCV1_0-cache
 EELAYER 25 0
@@
 F 0 "P2" H 5300 3775 50  0000 C CNN
 F 1 "CONN_02X08" V 5300 3325 50  0000 C CNN
-F 2 "" H 5300 2125 50  0001 C CNN
+F 2 "TP:Pin_Header_Straight_2x08" H 5300 2125 50  0001 C CNN
 F 3 "" H 5300 2125 50  0000 C CNN
 	1    5300 3325
@@
 $EndComp
 $Comp
-L GND #PWR09
+L GND #PWR08
 U 1 1 57993A55
 P 4825 2775
-F 0 "#PWR09" H 4825 2525 50  0001 C CNN
+F 0 "#PWR08" H 4825 2525 50  0001 C CNN
 F 1 "GND" H 4825 2625 50  0000 C CNN
 F 2 "" H 4825 2775 50  0000 C CNN
@@
 F 0 "RV1" H 3850 3225 50  0000 C CNN
 F 1 "POT" H 3850 3325 50  0000 C CNN
-F 2 "" H 3850 3325 50  0001 C CNN
+F 2 "TP:Connector_Molex_PicoBlade_53047-0310" H 3850 3325 50  0001 C CNN
 F 3 "" H 3850 3325 50  0000 C CNN
 	1    3850 3325
@@
 5V
 $Comp
-L GND #PWR010
+L GND #PWR09
 U 1 1 57993FAF
 P 3850 3675
-F 0 "#PWR010" H 3850 3425 50  0001 C CNN
+F 0 "#PWR09" H 3850 3425 50  0001 C CNN
 F 1 "GND" H 3850 3525 50  0000 C CNN
 F 2 "" H 3850 3675 50  0000 C CNN
@@
 F 0 "RV2" H 3850 4300 50  0000 C CNN
 F 1 "POT" H 3850 4400 50  0000 C CNN
-F 2 "" H 3850 4400 50  0001 C CNN
+F 2 "TP:Connector_Molex_PicoBlade_53047-0310" H 3850 4400 50  0001 C CNN
 F 3 "" H 3850 4400 50  0000 C CNN
 	1    3850 4400
@@
 5V
 $Comp
-L GND #PWR011
+L GND #PWR010
 U 1 1 57994190
 P 3850 4750
-F 0 "#PWR011" H 3850 4500 50  0001 C CNN
+F 0 "#PWR010" H 3850 4500 50  0001 C CNN
 F 1 "GND" H 3850 4600 50  0000 C CNN
 F 2 "" H 3850 4750 50  0000 C CNN
@@
 F 0 "R5" H 3375 3900 60  0000 C CNN
 F 1 "Res1206" H 3425 4225 60  0000 C CNN
-F 2 "TP:Resistor_SMD+THTuniversal_1206_RM10_HandSoldering_RevA_Date25Jun2010" H 3350 4025 60  0001 C CNN
+F 2 "TP:Resistor_SMD+THTuniversal_1206_RM10_HandSoldering" H 3350 4025 60  0001 C CNN
 F 3 "" H 3350 4025 60  0000 C CNN
 	1    3350 4025
