File: TP_IVAN_LEON/MCU.sch (KiCad schematic (older format))
At the start: 21 parts, among them P3 CONN_01X06, P4 POWER_OUT, P5 ANALOG_IN, U2 32.768HZ, U3 12MHZ, U4 LPC1769FBD100

Commit message: Acabado el pcb, aun no se agrega titulos a los sheets y falta completar cmapos de componenetes
Parts:
- C10, C11, C12, C9: footprint TP:c_1206 -> TP:C_0805_HandSoldering
- L3: footprint (none) -> TP:Choke_SMD_1206_Standard
- P3: footprint (none) -> TP:Connector_Molex_PicoBlade_53047-0610
- P4, P5: footprint (none) -> TP:Connector_Molex_PicoBlade_53047-0210
- R6: footprint TP:Resistor_SMD+THTuniversal_1206_RM10_HandSoldering_RevA_Date25Jun2010 -> TP:Resistor_SMD+THTuniversal_1206_RM10_HandSoldering
- R7: renamed from R?; footprint TP:Resistor_SMD+THTuniversal_1206_RM10_HandSoldering_RevA_Date25Jun2010 -> TP:Resistor_SMD+THTuniversal_1206_RM10_HandSoldering
- U2, U3: footprint TPun:Crystal_HC49-U_Horizontal_Typ1 -> TP:Crystal_HC49-U_Vertical
Connections:
- net GND: no longer C13.2, C14.2, C15.2, C16.2, C17.2, C18.2, C19.2, C20.2, L3.2, U4.28 (VDD(3V3)), U4.42 (VDD(REG)(3V3)), U4.54 (VDD(3V3)), U4.71 (VDD(3V3)), U4.84 (VDD(REG)(3V3)), U4.96 (VDD(3V3))
- net LCD1: now also U4.75 (P2[0]/PWM1[1]/TXD1); no longer U4.44 (P1[28]/MCOA2/PCAP1[0]/MAT0[0])
- net LCD2: now also U4.74 (P2[1]/PWM1[2]/RXD1); no longer U4.45 (P1[29]/MCOB2/PCAP1[1]/MAT0[1])
- net LCD3: now also U4.73 (P2[2]/PWM1[3]/CTS1/TRACEDATA[3]); no longer U4.21 (P1[30]/VBUS/AD0[4])
- net LCD4: now also U4.70 (P2[3]/PWM1[4]/DCD1/TRACEDATA[2]); no longer U4.20 (P1[31]/SCK1/AD0[5])
- net LCD5: now also U4.69 (P2[4]/PWM1[5]/DSR1/TRACEDATA[1]); no longer U4.75 (P2[0]/PWM1[1]/TXD1)
- net LCD6: now also U4.68 (P2[5]/PWM1[6]/DTR1/TRACEDATA[0]); no longer U4.74 (P2[1]/PWM1[2]/RXD1)
- net LCD7: now also U4.67 (P2[6]/PCAP1[0]/RI1/TRACECLK); no longer U4.73 (P2[2]/PWM1[3]/CTS1/TRACEDATA[3])
- net LCD8: now also U4.66 (P2[7]/RD2/RTS1); no longer U4.70 (P2[3]/PWM1[4]/DCD1/TRACEDATA[2])
- net Teclado1: now also U4.65 (P2[8]/TD2/TXD2); no longer U4.68 (P2[5]/PWM1[6]/DTR1/TRACEDATA[0])
- net Teclado2: now also U4.64 (P2[9]/USB_CONNECT/RXD2); no longer U4.67 (P2[6]/PCAP1[0]/RI1/TRACECLK)
- net Teclado3: now also U4.53 (P2[10]/~EINT0~/NMI); no longer U4.66 (P2[7]/RD2/RTS1)
- net Teclado4: now also U4.52 (P2[11]/~EINT1~/I2STX_CLK); no longer U4.65 (P2[8]/TD2/TXD2)
- net Teclado5: now also U4.51 (P2[12]/~EINT2~/I2STX_WS); no longer U4.64 (P2[9]/USB_CONNECT/RXD2)
- new net: C13.2, C14.2, C15.2, C16.2, C17.2, C18.2, C19.2, C20.2, L3.2, U4.28 (VDD(3V3)), U4.42 (VDD(REG)(3V3)), U4.54 (VDD(3V3)), U4.71 (VDD(3V3)), U4.84 (VDD(REG)(3V3)), U4.96 (VDD(3V3))
Changed lines of the file:
@@
 LIBS:MIproy1-cache
 LIBS:nxp_armmcu
+LIBS:DCV1_0-cach
 LIBS:DCV1_0-cache
 EELAYER 25 0
@@
 F 0 "R6" H 1600 1400 60  0000 C CNN
 F 1 "Res1206" H 1550 1725 60  0000 C CNN
-F 2 "TP:Resistor_SMD+THTuniversal_1206_RM10_HandSoldering_RevA_Date25Jun2010" H 1575 1525 60  0001 C CNN
+F 2 "TP:Resistor_SMD+THTuniversal_1206_RM10_HandSoldering" H 1575 1525 60  0001 C CNN
 F 3 "" H 1575 1525 60  0000 C CNN
 	1    1575 1525
@@
 F 0 "U3" H 1675 5425 60  0000 C CNN
 F 1 "12MHZ" H 1700 5875 60  0000 C CNN
-F 2 "TPun:Crystal_HC49-U_Horizontal_Typ1" H 1725 5650 60  0001 C CNN
+F 2 "TP:Crystal_HC49-U_Vertical" H 1725 5650 60  0001 C CNN
 F 3 "" H 1725 5650 60  0000 C CNN
 	1    1675 5650
@@
 F 0 "C11" H 1375 5175 30  0000 C CNN
 F 1 "18pF" H 1375 5350 30  0000 C CNN
-F 2 "TP:c_1206" H 1400 5275 60  0001 C CNN
+F 2 "TP:C_0805_HandSoldering" H 1400 5275 60  0001 C CNN
 F 3 "" H 1400 5275 60  0000 C CNN
 	1    1375 5275
@@
 F 0 "C12" H 1375 5900 30  0000 C CNN
 F 1 "18pF" H 1375 6075 30  0000 C CNN
-F 2 "TP:c_1206" H 1400 6000 60  0001 C CNN
+F 2 "TP:C_0805_HandSoldering" H 1400 6000 60  0001 C CNN
 F 3 "" H 1400 6000 60  0000 C CNN
 	1    1375 6000
@@
 $EndComp
 $Comp
-L GND #PWR012
+L GND #PWR011
 U 1 1 578ECBCC
 P 700 5725
-F 0 "#PWR012" H 700 5475 50  0001 C CNN
+F 0 "#PWR011" H 700 5475 50  0001 C CNN
 F 1 "GND" H 700 5575 50  0000 C CNN
 F 2 "" H 700 5725 50  0000 C CNN
@@
 F 0 "U2" H 1650 6450 60  0000 C CNN
 F 1 "32.768HZ" H 1675 6900 60  0000 C CNN
-F 2 "TPun:Crystal_HC49-U_Horizontal_Typ1" H 1700 6675 60  0001 C CNN
+F 2 "TP:Crystal_HC49-U_Vertical" H 1700 6675 60  0001 C CNN
 F 3 "" H 1700 6675 60  0000 C CNN
 	1    1650 6675
@@
 F 0 "C9" H 1350 6200 30  0000 C CNN
 F 1 "18pF" H 1350 6375 30  0000 C CNN
-F 2 "TP:c_1206" H 1375 6300 60  0001 C CNN
+F 2 "TP:C_0805_HandSoldering" H 1375 6300 60  0001 C CNN
 F 3 "" H 1375 6300 60  0000 C CNN
 	1    1350 6300
@@
 F 0 "C10" H 1350 6925 30  0000 C CNN
 F 1 "18pF" H 1350 7100 30  0000 C CNN
-F 2 "TP:c_1206" H 1375 7025 60  0001 C CNN
+F 2 "TP:C_0805_HandSoldering" H 1375 7025 60  0001 C CNN
 F 3 "" H 1375 7025 60  0000 C CNN
 	1    1350 7025
@@
 $EndComp
 $Comp
-L GND #PWR013
+L GND #PWR012
 U 1 1 578EDDB8
 P 675 6750
-F 0 "#PWR013" H 675 6500 50  0001 C CNN
+F 0 "#PWR012" H 675 6500 50  0001 C CNN
 F 1 "GND" H 675 6600 50  0000 C CNN
 F 2 "" H 675 6750 50  0000 C CNN
@@
 F 0 "L3" H 6400 1325 60  0000 C CNN
 F 1 "BK1608HS220-T" H 6375 1100 60  0000 C CNN
-F 2 "" H 6375 1200 60  0001 C CNN
+F 2 "TP:Choke_SMD_1206_Standard" H 6375 1200 60  0001 C CNN
 F 3 "" H 6375 1200 60  0000 C CNN
 	1    6375 1200
@@
 $EndComp
 $Comp
-L GND #PWR014
+L GND #PWR013
 U 1 1 57913828
 P 9150 2075
-F 0 "#PWR014" H 9150 1825 50  0001 C CNN
+F 0 "#PWR013" H 9150 1825 50  0001 C CNN
 F 1 "GND" H 9150 1925 50  0000 C CNN
 F 2 "" H 9150 2075 50  0000 C CNN
@@
 $EndComp
 $Comp
-L GND #PWR015
+L GND #PWR014
 U 1 1 5797E345
 P 5850 7075
-F 0 "#PWR015" H 5850 6825 50  0001 C CNN
+F 0 "#PWR014" H 5850 6825 50  0001 C CNN
 F 1 "GND" H 5850 6925 50  0000 C CNN
 F 2 "" H 5850 7075 50  0000 C CNN
@@
 Entry Wire Line
 	2300 2175 2400 2275
-Text HLabel 8250 4650 2    60   Input ~ 0
+Text HLabel 7900 5500 2    60   Input ~ 0
 Teclado[1..5]
 Entry Wire Line
+	7000 5300 7100 5400
+Entry Wire Line
 	7000 5000 7100 5100
 Entry Wire Line
-	7000 4700 7100 4800
-Entry Wire Line
-	7000 4800 7100 4900
-Entry Wire Line
-	7000 4900 7100 5000
-Text Label 6675 4700 0    40   ~ 0
+	7000 5100 7100 5200
+Entry Wire Line
+	7000 5200 7100 5300
+Text Label 6675 5000 0    40   ~ 0
 Teclado1
-Text Label 6675 4800 0    40   ~ 0
+Text Label 6675 5100 0    40   ~ 0
 Teclado2
-Text Label 6675 4900 0    40   ~ 0
+Text Label 6675 5200 0    40   ~ 0
 Teclado3
-Text Label 6675 5000 0    40   ~ 0
+Text Label 6675 5300 0    40   ~ 0
 Teclado4
 Entry Wire Line
-	7000 5100 7100 5200
-Text Label 6675 5100 0    40   ~ 0
+	7000 5400 7100 5500
+Text Label 6675 5400 0    40   ~ 0
 Teclado5
 Text Label 3925 1800 0    40   ~ 0
@@
 Wire Wire Line
 	9150 2075 9150 1925
-Connection ~ 9600 900
 Wire Wire Line
 	9975 1150 9600 1150
-Connection ~ 9600 1150
-Wire Wire Line
-	9600 2950 9600 900
 Wire Wire Line
 	10600 2950 10600 900
@@
 	2300 2175 1925 2175
 Wire Bus Line
-	7100 4650 7100 5100
-Wire Bus Line
-	7100 4650 8250 4650
-Wire Wire Line
-	7000 4700 6625 4700
-Wire Wire Line
-	6625 4800 7000 4800
-Wire Wire Line
-	7000 4900 6625 4900
-Wire Wire Line
-	6625 5000 7000 5000
-Wire Wire Line
-	7000 5100 6625 5100
-Wire Bus Line
-	7100 5075 7100 5200
+	7100 4950 7100 5400
+Wire Wire Line
+	7000 5000 6625 5000
+Wire Wire Line
+	6625 5100 7000 5100
+Wire Wire Line
+	7000 5200 6625 5200
+Wire Wire Line
+	6625 5300 7000 5300
+Wire Wire Line
+	7000 5400 6625 5400
+Wire Bus Line
+	7100 5375 7100 5525
 Wire Wire Line
 	4225 3850 3700 3850
 Wire Wire Line
+	6625 4700 7375 4700
+Wire Wire Line
+	6625 4800 7375 4800
+Wire Wire Line
+	6625 4900 7375 4900
+Wire Wire Line
+	6625 4600 7375 4600
+Wire Wire Line
+	6625 4500 7375 4500
+Wire Wire Line
+	6625 4400 7375 4400
+Wire Wire Line
+	6625 4200 7375 4200
+Wire Wire Line
 	6625 4300 7375 4300
-Wire Wire Line
-	6625 4400 7375 4400
-Wire Wire Line
-	6625 4500 7375 4500
-Wire Wire Line
-	6625 4200 7375 4200
-Wire Wire Line
-	6625 4000 7375 4000
-Wire Wire Line
-	6625 3900 7375 3900
-Wire Wire Line
-	6625 3700 7375 3700
-Wire Wire Line
-	6625 3800 7375 3800
-Entry Wire Line
-	7375 3700 7475 3800
-Entry Wire Line
-	7375 3800 7475 3900
-Entry Wire Line
-	7375 3900 7475 4000
-Entry Wire Line
-	7375 4000 7475 4100
 Entry Wire Line
 	7375 4200 7475 4300
@@
 	7375 4400 7475 4500
 Entry Wire Line
-	7375 4500 7475 4600
-Wire Bus Line
-	7475 4600 7475 3700
-Wire Bus Line
-	7475 3700 8200 3700
-Text HLabel 8200 3700 2    40   Input ~ 0
+	7375 4400 7475 4500
+Entry Wire Line
+	7375 4600 7475 4700
+Entry Wire Line
+	7375 4700 7475 4800
+Entry Wire Line
+	7375 4800 7475 4900
+Entry Wire Line
+	7375 4900 7475 5000
+Wire Bus Line
+	7475 5100 7475 4200
+Wire Bus Line
+	7475 4200 8200 4200
+Text HLabel 8200 4200 2    40   Input ~ 0
 LCD[1..8]
-Text Label 6700 3700 0    60   ~ 0
+Text Label 6700 4200 0    60   ~ 0
 LCD1
-Text Label 6700 3800 0    60   ~ 0
+Text Label 6700 4300 0    60   ~ 0
 LCD2
-Text Label 6700 3900 0    60   ~ 0
+Text Label 6700 4400 0    60   ~ 0
 LCD3
-Text Label 6700 4000 0    60   ~ 0
+Text Label 6700 4500 0    60   ~ 0
 LCD4
-Text Label 6725 4200 0    60   ~ 0
+Text Label 6725 4600 0    60   ~ 0
 LCD5
-Text Label 6725 4300 0    60   ~ 0
+Text Label 6725 4700 0    60   ~ 0
 LCD6
-Text Label 6725 4400 0    60   ~ 0
+Text Label 6725 4800 0    60   ~ 0
 LCD7
-Text Label 6725 4500 0    60   ~ 0
+Text Label 6725 4900 0    60   ~ 0
 LCD8
 Wire Wire Line
 	4225 4650 2750 4650
 $Comp
-L GND #PWR016
+L GND #PWR015
 U 1 1 5799B61F
 P 2925 4775
-F 0 "#PWR016" H 2925 4525 50  0001 C CNN
+F 0 "#PWR015" H 2925 4525 50  0001 C CNN
 F 1 "GND" H 2925 4625 50  0000 C CNN
 F 2 "" H 2925 4775 50  0000 C CNN
@@
 F 0 "P5" H 2550 4850 50  0000 C CNN
 F 1 "ANALOG_IN" V 2650 4700 50  0000 C CNN
-F 2 "" H 2550 4700 50  0001 C CNN
+F 2 "TP:Connector_Molex_PicoBlade_53047-0210" H 2550 4700 50  0001 C CNN
 F 3 "" H 2550 4700 50  0000 C CNN
 	1    2550 4700
@@
 F 0 "P4" H 2550 4375 50  0000 C CNN
 F 1 "POWER_OUT" V 2650 4225 50  0000 C CNN
-F 2 "" H 2550 4225 50  0001 C CNN
+F 2 "TP:Connector_Molex_PicoBlade_53047-0210" H 2550 4225 50  0001 C CNN
 F 3 "" H 2550 4225 50  0000 C CNN
 	1    2550 4225
@@
 NoConn ~ 6625 5700
 NoConn ~ 6625 5600
-NoConn ~ 6625 5400
-NoConn ~ 6625 5300
-NoConn ~ 6625 5200
 NoConn ~ 6625 1600
 NoConn ~ 6625 1700
@@
 F 0 "P3" H 1725 2375 50  0000 C CNN
 F 1 "CONN_01X06" V 1825 2025 50  0000 C CNN
-F 2 "" H 1725 2025 50  0001 C CNN
+F 2 "TP:Connector_Molex_PicoBlade_53047-0610" H 1725 2025 50  0001 C CNN
 F 3 "" H 1725 2025 50  0000 C CNN
 	1    1725 2025
@@
 Wire Wire Line
 	2000 2275 1925 2275
-NoConn ~ 6625 4600
-$Comp
-L Res1206 R?
+$Comp
+L Res1206 R7
 U 1 1 579AC0B2
 P 3325 6050
-F 0 "R?" H 3350 5925 60  0000 C CNN
+F 0 "R7" H 3350 5925 60  0000 C CNN
 F 1 "Res1206" H 3300 6250 60  0000 C CNN
-F 2 "TP:Resistor_SMD+THTuniversal_1206_RM10_HandSoldering_RevA_Date25Jun2010" H 3325 6050 60  0001 C CNN
+F 2 "TP:Resistor_SMD+THTuniversal_1206_RM10_HandSoldering" H 3325 6050 60  0001 C CNN
 F 3 "" H 3325 6050 60  0000 C CNN
 	1    3325 6050
@@
 Wire Wire Line
 	4225 6050 3650 6050
+Wire Wire Line
+	9600 1150 9600 2950
+Entry Wire Line
+	7375 4500 7475 4600
+Wire Bus Line
+	7100 5525 7900 5525
+Wire Bus Line
+	7900 5525 7900 5500
+NoConn ~ 6625 3700
+NoConn ~ 6625 3800
+NoConn ~ 6625 3900
+NoConn ~ 6625 4000
 $EndSCHEMATC
