File: TP_IVAN_LEON/MIDI.sch (KiCad schematic (older format))
At the start: 6 parts, among them P6 DIN_5

Commit message: Acabado el pcb, aun no se agrega titulos a los sheets y falta completar cmapos de componenetes
Parts:
- FB1: footprint (none) -> TP:Choke_SMD_1206_Standard
- L2: footprint TP:c_1206 -> TP:Choke_SMD_1206_Standard
- P6: footprint (none) -> TP:din-5
- R2, R4: footprint TP:Resistor_SMD+THTuniversal_1206_RM10_HandSoldering_RevA_Date25Jun2010 -> TP:Resistor_SMD+THTuniversal_1206_RM10_HandSoldering
- R3: footprint (none) -> TP:Resistor_SMD+THTuniversal_0805to2512_RM10_HandSoldering
Changed lines of the file:
@@
 LIBS:MIproy1-cache
 LIBS:nxp_armmcu
+LIBS:DCV1_0-cach
 LIBS:DCV1_0-cache
 EELAYER 25 0
@@
 F 0 "L2" H 6600 3150 60  0000 C CNN
 F 1 "100K@10MHZ" H 6575 2875 60  0000 C CNN
-F 2 "TP:c_1206" H 6575 2975 60  0001 C CNN
+F 2 "TP:Choke_SMD_1206_Standard" H 6575 2975 60  0001 C CNN
 F 3 "" H 6575 2975 60  0000 C CNN
 	1    6575 2975
@@
 F 0 "R3" H 3900 2850 60  0000 C CNN
 F 1 "Res0805" H 3950 3150 60  0000 C CNN
-F 2 "" H 3900 2975 60  0001 C CNN
+F 2 "TP:Resistor_SMD+THTuniversal_0805to2512_RM10_HandSoldering" H 3900 2975 60  0001 C CNN
 F 3 "" H 3900 2975 60  0000 C CNN
 	1    3900 2975
@@
 F 0 "R2" H 3225 2850 60  0000 C CNN
 F 1 "Res1206" H 3275 3175 60  0000 C CNN
-F 2 "TP:Resistor_SMD+THTuniversal_1206_RM10_HandSoldering_RevA_Date25Jun2010" H 3200 2975 60  0001 C CNN
+F 2 "TP:Resistor_SMD+THTuniversal_1206_RM10_HandSoldering" H 3200 2975 60  0001 C CNN
 F 3 "" H 3200 2975 60  0000 C CNN
 	1    3200 2975
@@
 F 0 "R4" H 7425 2850 60  0000 C CNN
 F 1 "Res1206" H 7475 3175 60  0000 C CNN
-F 2 "TP:Resistor_SMD+THTuniversal_1206_RM10_HandSoldering_RevA_Date25Jun2010" H 7400 2975 60  0001 C CNN
+F 2 "TP:Resistor_SMD+THTuniversal_1206_RM10_HandSoldering" H 7400 2975 60  0001 C CNN
 F 3 "" H 7400 2975 60  0000 C CNN
 	1    7400 2975
@@
 F 0 "P6" H 5600 2775 50  0000 C CNN
 F 1 "DIN_5" H 5600 2625 50  0000 C CNN
-F 2 "" H 5600 2775 50  0001 C CNN
+F 2 "TP:din-5" H 5600 2775 50  0001 C CNN
 F 3 "" H 5600 2775 50  0000 C CNN
 	1    5600 2775
@@
 F 0 "FB1" H 4725 3125 50  0000 C CNN
 F 1 "FILTER" H 4725 2875 50  0000 C CNN
-F 2 "" H 4725 2975 50  0001 C CNN
+F 2 "TP:Choke_SMD_1206_Standard" H 4725 2975 50  0001 C CNN
 F 3 "" H 4725 2975 50  0000 C CNN
 	1    4725 2975
